Commit message: Version 2; some corrections

File: config/arm.xacro (robot description, xacro)
@@ -1,4 +1,4 @@
 <?xml version="1.0" ?>
-<robot xmlns:xacro="http://www.ros.org/wiki/xacro" name="arm">
+<robot xmlns:xacro="http://www.ros.org/wiki/xacro" name="servoarm">
   <xacro:macro name="arm">
     <group name="arm">
@@ -34,4 +34,12 @@
       <joint name="top_joint" value="0.5" />
     </group_state>
+    <virtual_joint name="virtual_joint" type="floating" parent_frame="world" child_link="base_link" />
+    <disable_collisions link1="base_link" link2="platform" reason="Adjacent"/>
+    <disable_collisions link1="base_link" link2="lower_arm" reason="Never"/>
+    <disable_collisions link1="lower_arm" link2="platform" reason="Adjacent"/>
+    <disable_collisions link1="lower_arm" link2="wrist" reason="Never"/>
+    <disable_collisions link1="top_arm" link2="lower_arm" reason="Adjacent"/>
+    <disable_collisions link1="wrist" link2="top_arm" reason="Adjacent"/>
+    <disable_collisions link1="platform" link2="wrist" reason="Never"/>
   </xacro:macro>
 </robot>

File: config/hand.ros2_control.xacro (robot description, xacro)
@@ -1,6 +1,5 @@
 <?xml version="1.0"?>
 <robot xmlns:xacro="http://www.ros.org/wiki/xacro">
-    <xacro:macro name="hand_ros2_control"  params="name initial_positions_file ros2_control_hardware_type">
-    <xacro:property name="initial_positions" value="${xacro.load_yaml(initial_positions_file)['initial_positions']}"/>
+    <xacro:macro name="hand_ros2_control"  params="name ros2_control_hardware_type">
         <ros2_control name="${name}" type="system">
             <hardware>
@@ -14,4 +13,5 @@
                 </xacro:if>
             </hardware>
+	    <!--
             <joint name="hand_joint">
                 <command_interface name="position"/>
@@ -23,4 +23,5 @@
                 </state_interface>
             </joint>
+	    -->
             <joint name="clawl_joint">
                 <command_interface name="position"/>
@@ -28,7 +29,10 @@
                   <param name="initial_value">0.0</param>
                 </state_interface>
+		<!--
                 <state_interface name="velocity">
                         <param name="initial_value">0.0</param>
                 </state_interface>
+		-->
+                <state_interface name="velocity"/>
             </joint>
             <joint name="clawr_joint">
@@ -39,7 +43,10 @@
                   <param name="initial_value">0.0</param>
                 </state_interface>
+		<!--
                 <state_interface name="velocity">
                         <param name="initial_value">0.0</param>
                 </state_interface>
+		-->
+                <state_interface name="velocity"/>
             </joint>
         </ros2_control>

File: config/hand.xacro (robot description, xacro)
@@ -1,7 +1,6 @@
 <?xml version="1.0" ?>
-<robot xmlns:xacro="http://www.ros.org/wiki/xacro" name="arm">
+<robot xmlns:xacro="http://www.ros.org/wiki/xacro" name="servoarm">
   <xacro:macro name="hand">
     <group name="hand">
-        <joint name="hand_joint"/>
         <link name="clawbase"/>
         <link name="clawr"/>
@@ -9,4 +8,5 @@
         <joint name="clawl_joint"/>
         <passive_joint name="clawr_joint"/>
+        <joint name="hand_joint"/>
          <!--
         <chain base_link="eef_link" tip_link="clawl"/>

File: config/servoarm.srdf.xacro (robot description, xacro)
@@ -19,13 +19,9 @@
      <joint name="hand_joint" value="0" />
   </group_state>
-  <virtual_joint name="virtual_joint" type="floating" parent_frame="world" child_link="base_link" />
   <end_effector name="hand" parent_link="eef_link" group="hand" parent_group="arm" />
-    <disable_collisions link1="base_link" link2="lower_arm" reason="Never"/>
-    <disable_collisions link1="base_link" link2="platform" reason="Adjacent"/>
     <disable_collisions link1="clawbase" link2="lower_arm" reason="Never"/>
     <disable_collisions link1="clawbase" link2="platform" reason="Never"/>
     <disable_collisions link1="clawbase" link2="top_arm" reason="Never"/>
     <disable_collisions link1="clawbase" link2="wrist" reason="Adjacent"/>
-    <disable_collisions link1="clawl" link2="clawr" reason="Never"/>
     <disable_collisions link1="clawl" link2="lower_arm" reason="Never"/>
     <disable_collisions link1="clawl" link2="platform" reason="Never"/>
@@ -41,6 +37,3 @@
     <disable_collisions link1="platform" link2="wrist" reason="Never"/>
     <disable_collisions link1="top_arm" link2="wrist" reason="Adjacent"/>
-    <disable_collisions link1="clawbase" link2="clawr" reason="Adjacent" />
-    <disable_collisions link1="clawbase" link2="clawl" reason="Adjacent" />
-    <disable_collisions link1="clawr" link2="clawl" reason="Default" />
 </robot>

File: config/servoarm.urdf.xacro (robot description, xacro)
@@ -7,4 +7,4 @@
     <xacro:include filename="hand.ros2_control.xacro" />
     <xacro:arm_ros2_control name="ServoarmArmFakeSystem"   initial_positions_file="$(arg initial_positions_file)" ros2_control_hardware_type="$(arg ros2_control_hardware_type)"/>
-    <xacro:hand_ros2_control name="ServoarmHandFakeSystem" initial_positions_file="$(arg initial_positions_file)" ros2_control_hardware_type="$(arg ros2_control_hardware_type)"/>
+    <xacro:hand_ros2_control name="ServoarmHandFakeSystem" ros2_control_hardware_type="$(arg ros2_control_hardware_type)"/>
 </robot>

File: config/urdf/arm.urdf (robot description, URDF)
Before this commit: robot servoarm, 9 links, 8 joints
Joints:
- joint clawl_joint: type revolute -> prismatic
- joint clawr_joint: mimic joint=clawl_joint multiplier=-1 offset=0 -> joint=clawl_joint; type revolute -> prismatic

Commit message: version 5; minor changes

File: config/arm.xacro (robot description, xacro)
@@ -21,5 +21,5 @@
       <joint name="lower_joint" value="0.007" />
       <joint name="top_joint" value="0.007" />
-      <joint name="eef_joint" value="0.0" />
+      <joint name="eef_joint" value="0.007" />
     </group_state>
     <group_state name="pose1" group="arm">
@@ -28,5 +28,5 @@
       <joint name="lower_joint" value="0.017" />
       <joint name="top_joint" value="0.017" />
-      <joint name="eef_joint" value="0.0" />
+      <joint name="eef_joint" value="0.007" />
     </group_state>
     <group_state name="extended" group="arm">
@@ -35,5 +35,5 @@
       <joint name="lower_joint" value="0.5" />
       <joint name="top_joint" value="0.5" />
-      <joint name="eef_joint" value="0.0" />
+      <joint name="eef_joint" value="0.007" />
     </group_state>
     <virtual_joint name="virtual_joint" type="floating" parent_frame="world" child_link="base_link" />

File: config/hand.xacro (robot description, xacro)
@@ -8,8 +8,4 @@
         <joint name="clawl_joint"/>
         <passive_joint name="clawr_joint"/>
-         <!--
-        <joint name="hand_joint"/>
-        <chain base_link="eef_link" tip_link="clawl"/>
-	 -->
     </group>
     <disable_collisions link1="clawbase" link2="clawr" reason="Adjacent" />

File: config/servoarm.srdf.xacro (robot description, xacro)
@@ -10,15 +10,18 @@
   </group>
   <group_state name="open" group="hand">
-     <joint name="clawl_joint" value="0.035" />
-     <joint name="clawr_joint" value="0" />
+     <joint name="clawl_joint" value="0.4" />
+     <!--
+     <joint name="clawr_joint" value="-0.4" />
+     -->
   </group_state>
   <group_state name="close" group="hand">
      <joint name="clawl_joint" value="0" />
+     <!--
      <joint name="clawr_joint" value="0" />
-     <!--
      <joint name="hand_joint" value="0" />
      -->
   </group_state>
   <end_effector name="hand" parent_link="eef_link" group="hand" parent_group="arm" />
+    <disable_collisions link1="clawbase" link2="eef_link" reason="Never"/>
     <disable_collisions link1="clawbase" link2="lower_arm" reason="Never"/>
     <disable_collisions link1="clawbase" link2="platform" reason="Never"/>

File: config/urdf/arm.urdf (robot description, URDF)
Before this commit: robot servoarm, 9 links, 8 joints
Joints:
- joint clawr_joint: mimic joint=clawl_joint -> joint=clawl_joint multiplier=-1 offset=0
