Commit message: version4; eef_joint added

File: config/arm.ros2_control.xacro (robot description, xacro)
@@ -53,4 +53,13 @@
 	        </state_interface>
             </joint>
+            <joint name="eef_joint">
+                <command_interface name="position"/>
+                <state_interface name="position">
+                  <param name="initial_value">${initial_positions['eef_joint']}</param>
+                </state_interface>
+                <state_interface name="velocity">
+			<param name="initial_value">0.0</param>
+	        </state_interface>
+            </joint>
         </ros2_control>
     </xacro:macro>

File: config/arm.xacro (robot description, xacro)
@@ -17,8 +17,9 @@
     </group>
     <group_state name="ready" group="arm">
-      <joint name="base_joint" value="0.017" />
-      <joint name="platform_joint" value="0.017" />
-      <joint name="lower_joint" value="0.017" />
-      <joint name="top_joint" value="0.017" />
+      <joint name="base_joint" value="0.007" />
+      <joint name="platform_joint" value="0.007" />
+      <joint name="lower_joint" value="0.007" />
+      <joint name="top_joint" value="0.007" />
+      <joint name="eef_joint" value="0.0" />
     </group_state>
     <group_state name="pose1" group="arm">
@@ -27,4 +28,5 @@
       <joint name="lower_joint" value="0.017" />
       <joint name="top_joint" value="0.017" />
+      <joint name="eef_joint" value="0.0" />
     </group_state>
     <group_state name="extended" group="arm">
@@ -33,4 +35,5 @@
       <joint name="lower_joint" value="0.5" />
       <joint name="top_joint" value="0.5" />
+      <joint name="eef_joint" value="0.0" />
     </group_state>
     <virtual_joint name="virtual_joint" type="floating" parent_frame="world" child_link="base_link" />

File: config/hand.xacro (robot description, xacro)
@@ -8,6 +8,6 @@
         <joint name="clawl_joint"/>
         <passive_joint name="clawr_joint"/>
+         <!--
         <joint name="hand_joint"/>
-         <!--
         <chain base_link="eef_link" tip_link="clawl"/>
 	 -->

File: config/servoarm.srdf.xacro (robot description, xacro)
@@ -10,5 +10,4 @@
   </group>
   <group_state name="open" group="hand">
-     <joint name="hand_joint" value="0" />
      <joint name="clawl_joint" value="0.035" />
      <joint name="clawr_joint" value="0" />
@@ -17,5 +16,7 @@
      <joint name="clawl_joint" value="0" />
      <joint name="clawr_joint" value="0" />
+     <!--
      <joint name="hand_joint" value="0" />
+     -->
   </group_state>
   <end_effector name="hand" parent_link="eef_link" group="hand" parent_group="arm" />

File: config/urdf/arm.urdf (robot description, URDF)
Before this commit: robot servoarm, 9 links, 8 joints
Joints:
- joint clawl_joint: type prismatic -> revolute
- joint clawr_joint: type prismatic -> revolute
- joint eef_joint: axis 0 0 0 -> 0 1 0; limit (none) -> lower=-2.34 upper=2.34 effort=87 velocity=2.3925; type fixed -> revolute
- joint hand_joint: axis 0 1 0 -> 0 0 0; limit lower=-2.34 upper=2.34 effort=87 velocity=2.3925 -> (none); type revolute -> fixed

Commit message: version 6; minor changes

File: config/arm.ros2_control.xacro (robot description, xacro)
@@ -20,5 +20,5 @@
                 <command_interface name="position"/>
                 <state_interface name="position">
-                  <param name="initial_value">${initial_positions['platform_joint']}</param>
+                  <param name="initial_value">${initial_positions['base_joint']}</param>
                 </state_interface>
                 <state_interface name="velocity">

File: config/arm.xacro (robot description, xacro)
@@ -16,4 +16,25 @@
         <chain base_link="base_link" tip_link="eef_link"/>
     </group>
+    <group_state name="place" group="arm">
+      <joint name="base_joint" value="0.45378" />
+      <joint name="platform_joint" value="1.6580" />
+      <joint name="lower_joint" value="-2.14673" />
+      <joint name="top_joint" value="0.34906" />
+      <joint name="eef_joint" value="0.017" />
+    </group_state>
+    <group_state name="grasp" group="arm">
+      <joint name="base_joint" value="0.750483" />
+      <joint name="platform_joint" value="1.1344" />
+      <joint name="lower_joint" value="-1.8326" />
+      <joint name="top_joint" value="0.7854" />
+      <joint name="eef_joint" value="0.017" />
+    </group_state>
+    <group_state name="grasp_start" group="arm">
+      <joint name="base_joint" value="0.75049" />
+      <joint name="platform_joint" value="1.0" />
+      <joint name="lower_joint" value="0.017" />
+      <joint name="top_joint" value="0.017" />
+      <joint name="eef_joint" value="0.017" />
+    </group_state>
     <group_state name="ready" group="arm">
       <joint name="base_joint" value="0.007" />

Commit message: version 7; urdf and uros changes

File: config/arm.ros2_control.xacro (robot description, xacro)
@@ -1,7 +1,4 @@
 <?xml version="1.0"?>
 <robot xmlns:xacro="http://www.ros.org/wiki/xacro">
-	<!--
-    <xacro:arg name="initial_positions_file" default="initial_positions.yaml" />
-	-->
     <xacro:macro name="arm_ros2_control"  params="name initial_positions_file ros2_control_hardware_type">
     <xacro:property name="initial_positions" value="${xacro.load_yaml(initial_positions_file)['initial_positions']}"/>
@@ -11,8 +8,8 @@
                   <plugin>mock_components/GenericSystem</plugin>
                 </xacro:if>
-                <xacro:if value="${ros2_control_hardware_type == 'isaac'}">
+                <xacro:if value="${ros2_control_hardware_type == 'uros'}">
                     <plugin>topic_based_ros2_control/TopicBasedSystem</plugin>
-                    <param name="joint_commands_topic">/isaac_joint_commands</param>
-                    <param name="joint_states_topic">/isaac_joint_states</param>
+                    <param name="joint_commands_topic">/arm_joint_commands</param>
+                    <param name="joint_states_topic">/arm_joint_states</param>
                 </xacro:if>
             </hardware>

File: config/arm.xacro (robot description, xacro)
@@ -3,15 +3,4 @@
   <xacro:macro name="arm">
     <group name="arm">
-	    <!--
-        <link name="base_link"/>
-        <link name="platform"/>
-        <link name="lower_arm"/>
-        <link name="top_arm"/>
-        <link name="wrist"/>
-        <joint name="base_joint"/>
-        <joint name="platform_joint"/>
-        <joint name="lower_joint"/>
-        <joint name="top_joint"/>
-	    -->
         <chain base_link="base_link" tip_link="eef_link"/>
     </group>
@@ -19,5 +8,5 @@
       <joint name="base_joint" value="0.45378" />
       <joint name="platform_joint" value="1.6580" />
-      <joint name="lower_joint" value="-2.14673" />
+      <joint name="lower_joint" value="-1.954" />
       <joint name="top_joint" value="0.34906" />
       <joint name="eef_joint" value="0.017" />
@@ -59,11 +48,29 @@
     </group_state>
     <virtual_joint name="virtual_joint" type="floating" parent_frame="world" child_link="base_link" />
-    <disable_collisions link1="base_link" link2="platform" reason="Adjacent"/>
+    <disable_collisions link1="base_link" link2="base_link2" reason="Adjacent"/>
     <disable_collisions link1="base_link" link2="lower_arm" reason="Never"/>
-    <disable_collisions link1="lower_arm" link2="platform" reason="Adjacent"/>
+    <disable_collisions link1="base_link" link2="plate_bracket" reason="Never"/>
+    <disable_collisions link1="base_link" link2="plate_servo" reason="Never"/>
+    <disable_collisions link1="base_link" link2="platform_bracket" reason="Never"/>
+    <disable_collisions link1="base_link" link2="platform_servo" reason="Never"/>
+    <disable_collisions link1="base_link2" link2="plate_bracket" reason="Never"/>
+    <disable_collisions link1="base_link2" link2="plate_servo" reason="Never"/>
+    <disable_collisions link1="base_link2" link2="platform_bracket" reason="Adjacent"/>
+    <disable_collisions link1="base_link2" link2="platform_servo" reason="Never"/>
+    <disable_collisions link1="lower_arm" link2="plate_bracket" reason="Never"/>
+    <disable_collisions link1="lower_arm" link2="plate_servo" reason="Adjacent"/>
+    <disable_collisions link1="lower_arm" link2="top_arm" reason="Adjacent"/>
     <disable_collisions link1="lower_arm" link2="wrist" reason="Never"/>
-    <disable_collisions link1="top_arm" link2="lower_arm" reason="Adjacent"/>
-    <disable_collisions link1="wrist" link2="top_arm" reason="Adjacent"/>
-    <disable_collisions link1="platform" link2="wrist" reason="Never"/>
+    <disable_collisions link1="plate_bracket" link2="plate_servo" reason="Adjacent"/>
+    <disable_collisions link1="plate_bracket" link2="platform_bracket" reason="Never"/>
+    <disable_collisions link1="plate_bracket" link2="platform_servo" reason="Adjacent"/>
+    <disable_collisions link1="plate_bracket" link2="top_arm" reason="Never"/>
+    <disable_collisions link1="plate_bracket" link2="wrist" reason="Never"/>
+    <disable_collisions link1="plate_servo" link2="platform_bracket" reason="Never"/>
+    <disable_collisions link1="plate_servo" link2="platform_servo" reason="Never"/>
+    <disable_collisions link1="plate_servo" link2="top_arm" reason="Never"/>
+    <disable_collisions link1="plate_servo" link2="wrist" reason="Never"/>
+    <disable_collisions link1="platform_bracket" link2="platform_servo" reason="Adjacent"/>
+    <disable_collisions link1="top_arm" link2="wrist" reason="Adjacent"/>
   </xacro:macro>
 </robot>

File: config/hand.ros2_control.xacro (robot description, xacro)
@@ -1,5 +1,6 @@
 <?xml version="1.0"?>
 <robot xmlns:xacro="http://www.ros.org/wiki/xacro">
-    <xacro:macro name="hand_ros2_control"  params="name ros2_control_hardware_type">
+    <xacro:macro name="hand_ros2_control"  params="name initial_positions_file ros2_control_hardware_type">
+    <xacro:property name="initial_positions" value="${xacro.load_yaml(initial_positions_file)['initial_positions']}"/>
         <ros2_control name="${name}" type="system">
             <hardware>
@@ -7,15 +8,14 @@
                     <plugin>mock_components/GenericSystem</plugin>
                 </xacro:if>
-                <xacro:if value="${ros2_control_hardware_type == 'isaac'}">
+                <xacro:if value="${ros2_control_hardware_type == 'uros'}">
                     <plugin>topic_based_ros2_control/TopicBasedSystem</plugin>
-                    <param name="joint_commands_topic">/isaac_joint_commands</param>
-                    <param name="joint_states_topic">/isaac_joint_states</param>
+	            <param name="joint_commands_topic">/hand_joint_commands</param>
+                    <param name="joint_states_topic">/hand_joint_states</param>
                 </xacro:if>
             </hardware>
-	    <!--
-            <joint name="hand_joint">
+            <joint name="clawl_joint">
                 <command_interface name="position"/>
                 <state_interface name="position">
-                  <param name="initial_value">0.0</param>
+                  <param name="initial_value">${initial_positions['clawl_joint']}</param>
                 </state_interface>
                 <state_interface name="velocity">
@@ -23,17 +23,5 @@
                 </state_interface>
             </joint>
-	    -->
-            <joint name="clawl_joint">
-                <command_interface name="position"/>
-                <state_interface name="position">
-                  <param name="initial_value">0.0</param>
-                </state_interface>
-		<!--
-                <state_interface name="velocity">
-                        <param name="initial_value">0.0</param>
-                </state_interface>
-		-->
-                <state_interface name="velocity"/>
-            </joint>
+               <!--
             <joint name="clawr_joint">
                 <param name="mimic">clawl_joint</param>
@@ -41,13 +29,11 @@
                 <command_interface name="position" />
                 <state_interface name="position">
-                  <param name="initial_value">0.0</param>
+                  <param name="initial_value"> -${initial_positions['clawl_joint']}</param>
                 </state_interface>
-		<!--
                 <state_interface name="velocity">
                         <param name="initial_value">0.0</param>
                 </state_interface>
-		-->
-                <state_interface name="velocity"/>
             </joint>
+	       -->
         </ros2_control>
     </xacro:macro>

File: config/hand.xacro (robot description, xacro)
@@ -7,4 +7,7 @@
         <link name="clawl"/>
         <joint name="clawl_joint"/>
+	<!--
+        <joint name="clawr_joint"/>
+	-->
         <passive_joint name="clawr_joint"/>
     </group>

File: config/servoarm.srdf.xacro (robot description, xacro)
@@ -25,19 +25,11 @@
     <disable_collisions link1="clawbase" link2="eef_link" reason="Never"/>
     <disable_collisions link1="clawbase" link2="lower_arm" reason="Never"/>
-    <disable_collisions link1="clawbase" link2="platform" reason="Never"/>
     <disable_collisions link1="clawbase" link2="top_arm" reason="Never"/>
     <disable_collisions link1="clawbase" link2="wrist" reason="Adjacent"/>
     <disable_collisions link1="clawl" link2="lower_arm" reason="Never"/>
-    <disable_collisions link1="clawl" link2="platform" reason="Never"/>
     <disable_collisions link1="clawl" link2="top_arm" reason="Never"/>
     <disable_collisions link1="clawl" link2="wrist" reason="Never"/>
     <disable_collisions link1="clawr" link2="lower_arm" reason="Never"/>
-    <disable_collisions link1="clawr" link2="platform" reason="Never"/>
     <disable_collisions link1="clawr" link2="top_arm" reason="Never"/>
     <disable_collisions link1="clawr" link2="wrist" reason="Never"/>
-    <disable_collisions link1="lower_arm" link2="platform" reason="Adjacent"/>
-    <disable_collisions link1="lower_arm" link2="top_arm" reason="Adjacent"/>
-    <disable_collisions link1="lower_arm" link2="wrist" reason="Never"/>
-    <disable_collisions link1="platform" link2="wrist" reason="Never"/>
-    <disable_collisions link1="top_arm" link2="wrist" reason="Adjacent"/>
 </robot>

File: config/servoarm.urdf.xacro (robot description, xacro)
@@ -7,4 +7,4 @@
     <xacro:include filename="hand.ros2_control.xacro" />
     <xacro:arm_ros2_control name="ServoarmArmFakeSystem"   initial_positions_file="$(arg initial_positions_file)" ros2_control_hardware_type="$(arg ros2_control_hardware_type)"/>
-    <xacro:hand_ros2_control name="ServoarmHandFakeSystem" ros2_control_hardware_type="$(arg ros2_control_hardware_type)"/>
+    <xacro:hand_ros2_control name="ServoarmHandFakeSystem" initial_positions_file="$(arg initial_positions_file)" ros2_control_hardware_type="$(arg ros2_control_hardware_type)"/>
 </robot>

File: config/urdf/arm.urdf (robot description, URDF)
Before this commit: robot servoarm, 9 links, 8 joints
Links:
- removed link platform
- added link base_link2; collision mesh filename=package://armbot_moveit2/config/urdf/meshes/u_type_robot_wa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 scale=0.013 0.013 0.013; visual mesh filename=package://armbot_moveit2/config/urdf/meshes/u_type_robot_wa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 scale=0.013 0.013 0.013
- added link plate_bracket; collision mesh filename=package://armbot_moveit2/config/urdf/meshes/multi_functiona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 scale=0.013 0.013 0.013; visual mesh filename=package://armbot_moveit2/config/urdf/meshes/multi_functiona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 scale=0.013 0.013 0.013
- added link plate_servo; collision mesh filename=package://armbot_moveit2/config/urdf/meshes/mg996r_servo.stl scale=0.013 0.013 0.013; visual mesh filename=package://armbot_moveit2/config/urdf/meshes/mg996r_servo.stl scale=0.013 0.013 0.013
- added link platform_bracket; collision mesh filename=package://armbot_moveit2/config/urdf/meshes/multi_functiona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 scale=0.013 0.013 0.013; visual mesh filename=package://armbot_moveit2/config/urdf/meshes/multi_functiona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 scale=0.013 0.013 0.013
- added link platform_servo; collision mesh filename=package://armbot_moveit2/config/urdf/meshes/mg996r_servo.stl scale=0.013 0.013 0.013; visual mesh filename=package://armbot_moveit2/config/urdf/meshes/mg996r_servo.stl scale=0.013 0.013 0.013
- link base_link: geometry collision mesh filename=package://armbot_moveit2/config/urdf/meshes/u_type_robot_wa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 scale=0.013 0.013 0.013; visual mesh filename=package://armbot_moveit2/config/urdf/meshes/u_type_robot_wa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 scale=0.013 0.013 0.013
Joints:
- added joint base_joint_dummy: type fixed, parent base_link, child base_link2, origin xyz=0 0 0.0 rpy=0 0 0, axis 0 0 0
- added joint plate_servo_joint_dummy: type fixed, parent plate_bracket, child plate_servo, origin xyz=0 0 0.0 rpy=0 0 0, axis 0 0 0
- added joint platform_joint_dummy: type fixed, parent base_link2, child platform_bracket, origin xyz=0 0 0.0 rpy=0 0 0, axis 0 0 0
- added joint platform_servo_joint_dummy: type fixed, parent platform_bracket, child platform_servo, origin xyz=0 0 0.0 rpy=0 0 0, axis 0 0 0
- joint base_joint: child platform -> plate_bracket; limit lower=-2.34 upper=2.34 effort=87 velocity=2.3925 -> lower=-1.963 upper=1.963 effort=87 velocity=2.3925; origin xyz=0 0 0.48 rpy=0 0 0 -> xyz=0.115 -0.64 0.90 rpy=0 0 0; parent base_link -> platform_servo
- joint eef_joint: limit lower=-2.34 upper=2.34 effort=87 velocity=2.3925 -> lower=-1.963 upper=1.963 effort=87 velocity=2.3925
- joint lower_joint: limit lower=-2.34 upper=2.34 effort=87 velocity=2.3925 -> lower=-1.963 upper=1.963 effort=87 velocity=2.3925; origin xyz=-0.25 1.0 0 -> xyz=-0.23 1.02 0.015
- joint platform_joint: limit lower=-2.34 upper=2.34 effort=87 velocity=2.3925 -> lower=-1.963 upper=1.963 effort=87 velocity=2.3925; origin xyz=0 0.19 0.28 -> xyz=-0.045 -0.125 0.055 rpy=2.4 0 0; parent platform -> plate_servo
- joint top_joint: limit lower=-2.34 upper=2.34 effort=87 velocity=2.3925 -> lower=-1.963 upper=1.963 effort=87 velocity=2.3925; origin xyz=0.11 1.25 0 -> xyz=0.09 1.25 0
