Commit message: version 8; more changes;

File: config/servoarm.srdf.xacro (robot description, xacro)
@@ -10,15 +10,8 @@
   </group>
   <group_state name="open" group="hand">
-     <joint name="clawl_joint" value="0.4" />
-     <!--
-     <joint name="clawr_joint" value="-0.4" />
-     -->
+     <joint name="clawl_joint" value="0.62" />
   </group_state>
   <group_state name="close" group="hand">
-     <joint name="clawl_joint" value="0" />
-     <!--
-     <joint name="clawr_joint" value="0" />
-     <joint name="hand_joint" value="0" />
-     -->
+     <joint name="clawl_joint" value="1.57" />
   </group_state>
   <end_effector name="hand" parent_link="eef_link" group="hand" parent_group="arm" />

File: config/urdf/arm.urdf (robot description, URDF)
Before this commit: robot servoarm, 13 links, 12 joints
Joints:
- joint base_joint_dummy: origin xyz=0 0 0.0 rpy=0 0 0 -> xyz=0 0 0.0 rpy=0 0 0.0
- joint clawl_joint: axis 0 0 1 -> 0 0 -1; limit lower=0.0 upper=0.4 effort=87 velocity=0.2 -> lower=0.611 upper=1.57 effort=87 velocity=2.3925; origin xyz=-0.142 0.305 -0.05 rpy=0 0 0.31 -> xyz=-0.142 0.305 -0.05 rpy=0 0 1.77
- joint clawr_joint: axis 0 0 1 -> 0 0 -1; limit lower=-0.4 upper=0.0 effort=87 velocity=0.2 -> lower=-1.57 upper=-0.611 effort=87 velocity=2.3925; origin xyz=0.152 0.305 -0.05 rpy=0 0 -0.31 -> xyz=0.152 0.305 -0.05 rpy=0 0 -1.97
- joint lower_joint: origin xyz=-0.23 1.02 0.015 -> xyz=-0.23 1.02 0.015 rpy=-0.35 0 0
- joint platform_joint: axis 1 0 0 -> -1 0 0; origin xyz=-0.045 -0.125 0.055 rpy=2.4 0 0 -> xyz=-0.045 -0.125 0.055 rpy=1.95 0 0
- joint top_joint: axis 1 0 0 -> -1 0 0; origin xyz=0.09 1.25 0 -> xyz=0.09 1.25 0 rpy=-0.218 0 0
